File: modbus-pir-2servos/modbus-pir-2servos.kicad_sch (KiCad schematic)
At the start: 94 parts, among them J1 USB_B_Micro, J2 Conn_01x02, J4 Conn_02x10_Odd_Even, J5 Conn_01x02, J6 Conn_01x04, M1 Motor_Servo, M2 Motor_Servo, Q2 Q_PMOS_GSD, Q3 MMBT3904, SW1 RESET, SW2 USB_BOOT, U1 SP3485EN, U11 Logo, U2 LMR16030S, U3 RP2040, U4 HT75xx-1-SOT89, U5 PIR_P924M-S, U6 PIR_P924M-S, U7 PCF8563T, U8 LMR14050S, U9 W25Q128JVS, Y1 Crystal_GND24, Y2 Crystal

Commit message: Fix small issues
Parts:
- removed D11, D16: D_Shockley, Diode_SMD:D_SOD-323, symbol Device:D_Shockley
- removed D2: D_Shockley, Diode_SMD:D_SMA, symbol Device:D_Shockley
- removed J4: Conn_02x10_Odd_Even, Connector_PinSocket_2.54mm:PinSocket_2x07_P2.54mm_Vertical, symbol Connector_Generic:Conn_02x07_Odd_Even
- removed J6: Conn_01x04, Connector_JST:JST_XA_S04B-XASK-1_1x04_P2.50mm_Horizontal, symbol Connector_Generic:Conn_01x04
- removed JP1: Jumper_3_Open, Connector_PinSocket_2.54mm:PinSocket_1x03_P2.54mm_Vertical, symbol Jumper:Jumper_3_Open
- removed M1, M2: Motor_Servo, Connector_JST:JST_XA_S03B-XASK-1_1x03_P2.50mm_Horizontal, symbol Motor:Motor_Servo
- removed Q3: MMBT3904, Package_TO_SOT_SMD:SOT-23, symbol Transistor_BJT:MMBT3904
- added BZ1: Buzzer, cacophony-footprints:BUZ-TH_BD9.0-P5.00-D0.6-FD, symbol Device:Buzzer
- added D2, D3: D, Diode_SMD:D_SOD-123F, symbol Device:D
- added H4: MountingHole_Pad, MountingHole:MountingHole_3.2mm_M3_Pad, symbol Mechanical:MountingHole_Pad
- added J3: Conn_01x05, Connector_JST:JST_XA_B05B-XASK-1-A_1x05_P2.50mm_Vertical, symbol Connector_Generic:Conn_01x05
- added J4: Conn_02x05_Odd_Even, Connector_PinHeader_2.54mm:PinHeader_2x05_P2.54mm_Vertical, symbol Connector_Generic:Conn_02x05_Odd_Even
- added J6: Conn_01x02, Connector_PinSocket_2.54mm:PinSocket_1x02_P2.54mm_Vertical, symbol Connector_Generic:Conn_01x02
- added M1, M2: Servo, Connector_JST:JST_XA_B03B-XASK-1-A_1x03_P2.50mm_Vertical, symbol cacophony-symbols:Servo
- added Q1: 2N7002, Package_TO_SOT_SMD:SOT-23, symbol Transistor_FET:2N7002
- added SW3: SW_Coded_SH-7010, cacophony-footprints:SW-TH_6P-L10.0-W10.0-P2.54-LS7.6_TSR-10, symbol Switch:SW_Coded_SH-7010
- added SW4: SW_Push_DPDT, cacophony-footprints:SW-TH_K3-2235D-F1, symbol Switch:SW_Push_DPDT
- J1: footprint cacophony-footprints:920-E52A2021S10100 -> cacophony-footprints:MICRO-USB-TH_MICRO-USB-A14; LCSC C10418 -> C145795
- J2: footprint Connector_JST:JST_XA_S02B-XASK-1_1x02_P2.50mm_Horizontal -> Connector_JST:JST_XA_B02B-XASK-1-A_1x02_P2.50mm_Vertical; LCSC C225470 -> C265077
- J5, R10, U11: now left out of the parts list
- R1: value 100k -> 10k; LCSC C25086 -> C25744
- R19, R25: LCSC C25086 -> C25741
- R2: value 100k -> 100R; LCSC C25086 -> C25076
- U8: LCSC C136648 -> C155484
Connections:
- net GPIO13 is gone; now on net 6V_Enable: U3.16 (GPIO13)
- net GPIO22 is gone; now on net PIR_1: U3.34 (GPIO22)
- net PIR_4 is gone; now on net PIR_2: U3.32 (GPIO21)
- net ~{RE RP2040} is gone; now on net ~{RE}: U3.4 (GPIO2)
- net +3V3: now also BZ1.1 (-), D2.2 (A), J4.2 (Pin_2); no longer R2.2
- net +6V: now also M1.2 (+Ve), M2.2 (+Ve)
- net +ve: now also J3.2 (Pin_2)
- net 6V_Enable: no longer U3.14 (GPIO11)
- net DE: now also U3.5 (GPIO3), J6.2 (Pin_2); no longer R2.1
- net GND: now also J3.1 (Pin_1), J4.1 (Pin_1), J4.3 (Pin_3), M1.1 (GND), M2.1 (GND), Q1.2 (S), SW3.C, SW4.3 (C)
- net GPIO10: now also J4.5 (Pin_5)
- net GPIO12: now also J4.9 (Pin_9)
- net GPIO6: now also J4.4 (Pin_4)
- net GPIO7: now also J4.6 (Pin_6)
- net GPIO8: now also J4.8 (Pin_8)
- net GPIO9: now also J4.10 (Pin_10)
- net PIR_1: no longer U3.29 (GPIO18)
- net PIR_2: no longer U3.30 (GPIO19)
- net RS485_A: now also J3.3 (Pin_3)
- net RS485_B: now also J3.4 (Pin_4)
- net TX: no longer R1.1
- net ~{RE}: now also J6.1 (Pin_1)
- net at C9.1, U7.8 (VDD): now also D2.1 (K), D3.1 (K)
- net at R7.2: now also M2.3 (SIG)
- net at R1.2: now also BT1.1 (+), D3.2 (A)
- net at R6.2: now also M1.3 (SIG)
- net GPIO17 renamed R_ENC_4
- net R_ENC_4: now also SW3.4
- net GPIO26_ADC0 renamed RTC_BAT
- net RTC_BAT: now also R1.1
- net GPIO5 renamed BUZZER
- net BUZZER: now also Q1.1 (G)
- net IR_LED_ENABLE renamed R_ENC_1
- net R_ENC_1: now also SW3.1
- net PIR_3 renamed 24_hour
- net 24_hour: now also SW4.2 (B)
- new net: Q1.3 (D), R2.2
- new net: BZ1.2 (+), R2.1
- new net GPIO11: J4.7 (Pin_7), U3.14 (GPIO11)
- new net INTERRUPT: J3.5 (Pin_5)
- new net R_ENC_2: SW3.2, U3.29 (GPIO18)
- new net R_ENC_8: SW3.8, U3.30 (GPIO19)
- no-connect marks 7 -> 12
Other:
- note added: "TODO: - Fix 1 ohm resistors"
- note removed: "TODO: - Add buzzer?"
- moved on the sheet: C1, C2, C24, C26, C27, C28, C29, C3, C30, C31, C32, C33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

Commit message: WIP
Parts:
- removed BT1: Battery_Cell, cacophony-footprints:CR1220, symbol Device:Battery_Cell
- removed BZ1: Buzzer, cacophony-footprints:BUZ-TH_BD9.0-P5.00-D0.6-FD, symbol Device:Buzzer
- removed C1, C26: 220uF, cacophony-footprints:CAP-SMD_BD8.0-L8.3-W8.3-LS9.3-FD, symbol Device:C_Polarized_Small
- removed C2, C27, C28, C3: 2.2uF, Capacitor_SMD:C_0805_2012Metric, symbol Device:C_Small
- removed C24, C33, C34, C8: 47uF, Capacitor_SMD:C_1206_3216Metric, symbol Device:C_Small
- removed C29, C4: 470nF, Capacitor_SMD:C_0603_1608Metric, symbol Device:C_Small
- removed C30: 22nF, Capacitor_SMD:C_0402_1005Metric, symbol Device:C_Small
- removed C31: 100nF, Capacitor_SMD:C_0603_1608Metric, symbol Device:C
- removed C5: 10nF, Capacitor_SMD:C_0402_1005Metric, symbol Device:C_Small
- removed C6: 100nF, Capacitor_SMD:C_0603_1608Metric, symbol Device:C_Small
- removed C7: 1uF, Capacitor_SMD:C_0402_1005Metric, symbol Device:C_Small
- removed D1, D17: D_Shockley, Diode_SMD:D_SMA, symbol Device:D_Shockley
- removed D12: D_Zener, Diode_SMD:D_MiniMELF, symbol Device:D_Zener
- removed D13: LED, LED_SMD:LED_0805_2012Metric, symbol Device:LED
- removed D3: D, Diode_SMD:D_SOD-123F, symbol Device:D
- removed J2: Conn_01x02, Connector_JST:JST_XA_B02B-XASK-1-A_1x02_P2.50mm_Vertical, symbol Connector_Generic:Conn_01x02
- removed J3: Conn_01x05, Connector_JST:JST_XA_B05B-XASK-1-A_1x05_P2.50mm_Vertical, symbol Connector_Generic:Conn_01x05
- removed J4: Conn_02x05_Odd_Even, Connector_PinHeader_2.54mm:PinHeader_2x05_P2.54mm_Vertical, symbol Connector_Generic:Conn_02x05_Odd_Even
- removed J5, J6: Conn_01x02, Connector_PinSocket_2.54mm:PinSocket_1x02_P2.54mm_Vertical, symbol Connector_Generic:Conn_01x02
- removed L1: 15uH, cacophony-footprints:IND-SMD_L6.0-W6.0_SWPA6045S, symbol pspice:INDUCTOR
- removed L2: 4.7uH, cacophony-footprints:IND-SMD_L7.0-W6.6, symbol Device:L
- removed M1, M2: Servo, Connector_JST:JST_XA_B03B-XASK-1-A_1x03_P2.50mm_Vertical, symbol cacophony-symbols:Servo
- removed Q1: 2N7002, Package_TO_SOT_SMD:SOT-23, symbol Transistor_FET:2N7002
- removed Q2: Q_PMOS_GSD, Package_TO_SOT_SMD:SOT-23, symbol Device:Q_PMOS_GSD
- removed R14: 33k, Resistor_SMD:R_0603_1608Metric, symbol Device:R
- removed R15: 100k, Resistor_SMD:R_0603_1608Metric, symbol Device:R
- removed R16: 270k, Resistor_SMD:R_0603_1608Metric, symbol Device:R
- removed R17, R5: 47k, Resistor_SMD:R_0402_1005Metric, symbol Device:R
- removed R18: 10K, Resistor_SMD:R_0402_1005Metric, symbol Device:R
- removed R2: 100R, Resistor_SMD:R_0402_1005Metric, symbol Device:R
- removed R22, R6, R7: 1K, Resistor_SMD:R_0402_1005Metric, symbol Device:R
- removed R25: 100k, Resistor_SMD:R_0402_1005Metric, symbol Device:R
- removed R26: 560, Resistor_SMD:R_0603_1608Metric, symbol Device:R
- removed R27: 680, Resistor_SMD:R_0603_1608Metric, symbol Device:R
- removed R8: 82K, Resistor_SMD:R_0603_1608Metric, symbol Device:R
- removed RV1: R_Potentiometer, Potentiometer_SMD:Potentiometer_Bourns_TC33X_Vertical, symbol Device:R_Potentiometer
- removed SW3: SW_Coded_SH-7010, cacophony-footprints:SW-TH_6P-L10.0-W10.0-P2.54-LS7.6_TSR-10, symbol Switch:SW_Coded_SH-7010
- removed SW4: SW_Push_DPDT, cacophony-footprints:SW-TH_K3-2235D-F1, symbol Switch:SW_Push_DPDT
- removed U1: SP3485EN, Package_SO:SOIC-8_3.9x4.9mm_P1.27mm, symbol Interface_UART:SP3485EN
- removed U2: LMR16030S, Package_SO:TI_SO-PowerPAD-8, symbol cacophony-symbols:LMR16030S
- removed U4: HT75xx-1-SOT89, Package_TO_SOT_SMD:SOT-89-3, symbol Regulator_Linear:HT75xx-1-SOT89
- removed U5, U6: PIR_P924M-S, cacophony-footprints:PIR_P924M-S, symbol cacophony-symbols:PIR_P924M-S
- removed U8: LMR14050S, Package_SO:TI_SO-PowerPAD-8, symbol cacophony-symbols:LMR14050S
- added BT2: Battery_Cell, cacophony-library:CAP-SMD_FL11E, symbol Device:Battery_Cell
- added C38: 22pF, Capacitor_SMD:C_0402_1005Metric, symbol Device:C_Small
- added D4: D, Diode_SMD:D_SOD-523, symbol Device:D
- added J10: Conn_01x02, Connector_PinHeader_2.00mm:PinHeader_1x02_P2.00mm_Vertical, symbol Connector_Generic:Conn_01x02
- added J3, J8: Conn_02x03_Odd_Even, Connector_PinHeader_2.54mm:PinHeader_2x03_P2.54mm_Vertical, symbol Connector_Generic:Conn_02x03_Odd_Even
- added J6: SWD, Connector_PinHeader_2.54mm:PinHeader_1x03_P2.54mm_Vertical, symbol Connector_Generic:Conn_01x03
- added JP1: SolderJumper_2_Bridged, Jumper:SolderJumper-2_P1.3mm_Bridged_RoundedPad1.0x1.5mm, symbol Jumper:SolderJumper_2_Bridged
- added R13, R21, R23, R28, R30, R31, R33, R34, R35: 1k, Resistor_SMD:R_0402_1005Metric, symbol Device:R
- C10, C15: value 1u -> 1uF
- C23: symbol Device:C -> Device:C_Small
- C32: value 1uF -> 22pF; LCSC C52923 -> C1555
- H1, H2, H3, H4: footprint MountingHole:MountingHole_3.2mm_M3_Pad -> cacophony-library:MountingHole_3.2mm_M3; symbol Mechanical:MountingHole_Pad -> Mechanical:MountingHole; now left out of the parts list
- J1: footprint cacophony-footprints:MICRO-USB-TH_MICRO-USB-A14 -> cacophony-library:MICRO-USB-TH_MICRO-USB-A14
- R1: value 10k -> 1k; LCSC C25744 -> C11702
- R19: value 100k -> 1k; LCSC C25741 -> C11702
- R20: value 120R -> 1k; LCSC C25079 -> C11702
- R3, R4: value 27R -> 33ohm; footprint Resistor_SMD:R_0603_1608Metric -> Resistor_SMD:R_0402_1005Metric; LCSC C25190 -> C25105
- R9: value 1K -> 1k
- U11: footprint cacophony-footprints:logo -> cacophony-library:logo; symbol cacophony-symbols:Logo -> cacophony-library:Logo
- U3: footprint cacophony-footprints:RP2040-QFN-56 -> cacophony-library:RP2040-QFN-56; symbol cacophony-symbols:RP2040 -> cacophony-library:RP2040
Connections:
- net +6V is gone; now on an unnamed net: C32.1
- net 24_hour is gone; now on net R_ENC_8: U3.31 (GPIO20)
- net DE is gone; now on net SERVO_1_PHY: U3.5 (GPIO3)
- net GPIO10 is gone; now on an unnamed net: U3.13 (GPIO10)
- net GPIO12 is gone; now on net PIR_1: U3.15 (GPIO12)
- net RS485_A is gone; now on net SERVO_2_PHY: R20.1
- net +3V3: now also J3.5 (Pin_5), J8.2 (Pin_2)
- net BUZZER: now also U3.28 (GPIO17); no longer U3.7 (GPIO5)
- net GND: now also BT2.2 (-), C38.2, J3.1 (Pin_1), J3.3 (Pin_3), J6.2 (Pin_2), J8.1 (Pin_1), J8.3 (Pin_3), J8.5 (Pin_5); no longer R19.2
- net GPIO27_ADC1: now also J8.4 (Pin_4)
- net GPIO28_ADC2: now also J8.6 (Pin_6)
- net PIR_1: no longer U3.34 (GPIO22)
- net PIR_2: now also U3.27 (GPIO16); no longer U3.32 (GPIO21)
- net RTC_BAT: now also D4.1 (K), J10.2 (Pin_2), JP1.2 (B), R23.2; no longer R1.1, U3.38 (GPIO26_ADC0)
- net R_ENC_1: now also U3.32 (GPIO21); no longer U3.27 (GPIO16)
- net R_ENC_4: now also U3.30 (GPIO19); no longer U3.28 (GPIO17)
- net R_ENC_8: no longer U3.30 (GPIO19)
- net SERVO_1: now also R1.1; no longer U3.18 (GPIO15)
- net SERVO_2: now also R30.2; no longer U3.17 (GPIO14)
- net SWCLK: now also J6.3 (Pin_3)
- net SWD: now also J6.1 (Pin_1)
- net USB_D+: now also R3.2; no longer R3.1
- net USB_D-: now also R4.2; no longer R4.1
- net SERVO_1_PHY: now reaches R1.2
- net at U7.2 (OSCO), Y2.1: now also C38.1
- net RTC_V_{DD}: now reaches C9.1, D2.1 (K), U7.8 (VDD)
- net RTC_V_{DD}: now also R23.1
- net RP2040_TX_OUT_PHY: now reaches U3.6 (GPIO4)
- net RP2040_TX_OUT_PHY: now also R33.1
- net USB_PHY_D-: now reaches U3.46 (USB_DM)
- net USB_PHY_D-: now also R4.1; no longer R4.2
- net USB_PHY_D+: now reaches U3.47 (USB_DP)
- net USB_PHY_D+: now also R3.1; no longer R3.2
- net USB_BOOT: now reaches R9.2, SW2.2
- net 6V_Enable renamed GPIO13
- net GPIO13: now also J3.2 (Pin_2)
- net GPIO11: no longer names the net of U3.14 (GPIO11)
- net GPIO11: now also R35.1
- net GPIO29_ADC3 renamed RTC_BAT_SENSE_PHY
- net RTC_BAT_SENSE_PHY: now also R21.2
- net GPIO6 renamed LED_1_PHY
- net GPIO7 renamed SERVO_2_PHY
- net GPIO8 renamed 6V_EN_PHY
- net 6V_EN_PHY: now also R30.1
- net GPIO9: no longer names the net of U3.12 (GPIO9)
- net GPIO9: now also R34.1
- net RS485_B renamed SERVO_2_EN
- net RX renamed RP2040_RX_IN
- net TX renamed RP2040_TX_IN_PHY
- net RP2040_TX_IN_PHY: now also R31.1
- net ~{RE} renamed SERVO_1_EN_PHY
- net SERVO_1_EN_PHY: now also R13.1
- new net: BT2.1 (+), J10.1 (Pin_1), JP1.1 (A)
- new net 6V_EN: R35.2
- new net GPIO14: J3.4 (Pin_4), U3.17 (GPIO14)
- new net GPIO15: J3.6 (Pin_6), U3.18 (GPIO15)
- new net NIGHT_ONLY: U3.34 (GPIO22)
- new net PIR_SENS_POT: R28.2
- new net PIR_SENS_POT_FB: R28.1, U3.38 (GPIO26_ADC0)
- new net RP2040_RX_OUT: U3.7 (GPIO5)
- new net RP2040_TX_IN: R31.2
- new net RP2040_TX_OUT: R33.2
- new net RTC_BAT_SENSE: D4.2 (A), R21.1
- new net SERVO_1_EN: R13.2
- new net SWITCH_1: R34.2
- new net SWITCH_2: R19.2
- no-connect marks 12 -> 3
Other:
- added sheet input-output (input-output.kicad_sch)
- added sheet power (power.kicad_sch)
- note added: "RP2040 should setup with a pullup resistor"
- moved on the sheet: C10, C11, C12, C13, C14, C15, C16, C17, C18, C19, C20, C21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
