File: modbus-pir-2servos/input-output.kicad_sch (KiCad schematic)
At the start: 30 parts, among them J2 Switch_2, J4 Switch_1, J5 Switch_1, J7 Switch_1, J9 Conn_01x08, M1 Servo, M2 Servo, Q1 2N7002, Q3 Q_PMOS_GSD, Q4 2N7002, Q5 Q_PMOS_GSD, Q6 2N7002, SW3 SW_Coded_SH-7010, SW4 SW_Push_DPDT, SW5 SW_Push_DPDT, U1 TPL0401B-10-Q1, U5 PIR_P924M-S, U6 PIR_P924M-S

Commit message: WIP
Other:
- moved on the sheet: J4, J5
Changed lines of the file:
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@@
 	(wire
 		(pts
-			(xy 105.41 106.68) (xy 106.68 106.68)
+			(xy 102.87 106.68) (xy 104.14 106.68)
 		)
 		(stroke
@@
 	(wire
 		(pts
-			(xy 99.06 123.19) (xy 100.33 123.19)
+			(xy 102.87 123.19) (xy 104.14 123.19)
 		)
 		(stroke
@@
 	(wire
 		(pts
-			(xy 133.35 163.83) (xy 133.35 170.18)
+			(xy 133.35 165.1) (xy 133.35 170.18)
 		)
 		(stroke
@@
 	(wire
 		(pts
-			(xy 100.33 125.73) (xy 100.33 127)
+			(xy 104.14 125.73) (xy 104.14 127)
 		)
 		(stroke
@@
 	(wire
 		(pts
-			(xy 105.41 104.14) (xy 106.68 104.14)
+			(xy 102.87 104.14) (xy 104.14 104.14)
 		)
 		(stroke
@@
 	(wire
 		(pts
-			(xy 99.06 125.73) (xy 100.33 125.73)
+			(xy 102.87 125.73) (xy 104.14 125.73)
 		)
 		(stroke
@@
 	(wire
 		(pts
-			(xy 106.68 106.68) (xy 106.68 107.95)
+			(xy 104.14 106.68) (xy 104.14 107.95)
 		)
 		(stroke
@@
 	(wire
 		(pts
-			(xy 132.08 163.83) (xy 133.35 163.83)
+			(xy 132.08 165.1) (xy 133.35 165.1)
 		)
 		(stroke
@@
 	(text_box "SENS range from 0V to 0.25*V_{SS}"
 		(exclude_from_sim no)
-		(at 140.97 158.75 0)
+		(at 137.16 158.75 0)
 		(size 19.05 6.35)
 		(stroke
@@
 	(global_label "PIR_SENS_POT"
 		(shape input)
-		(at 132.08 163.83 180)
+		(at 132.08 165.1 180)
 		(fields_autoplaced yes)
 		(effects
@@
 		)
 		(property "Intersheetrefs" "${INTERSHEET_REFS}"
-			(at 115.5482 163.83 0)
+			(at 115.5482 165.1 0)
 			(effects
 				(font
@@
 	(global_label "SWITCH_2"
 		(shape input)
-		(at 100.33 123.19 0)
+		(at 104.14 123.19 0)
 		(fields_autoplaced yes)
 		(effects
@@
 		)
 		(property "Intersheetrefs" "${INTERSHEET_REFS}"
-			(at 112.3261 123.19 0)
+			(at 116.1361 123.19 0)
 			(effects
 				(font
@@
 	(global_label "SWITCH_1"
 		(shape input)
-		(at 106.68 104.14 0)
+		(at 104.14 104.14 0)
 		(fields_autoplaced yes)
 		(effects
@@
 		)
 		(property "Intersheetrefs" "${INTERSHEET_REFS}"
-			(at 118.6761 104.14 0)
+			(at 116.1361 104.14 0)
 			(effects
 				(font
@@
 	(symbol
 		(lib_id "power:GND")
-		(at 100.33 127 0)
+		(at 104.14 127 0)
 		(unit 1)
 		(exclude_from_sim no)
@@
 		(fields_autoplaced yes)
 		(property "Reference" "#PWR013"
-			(at 100.33 133.35 0)
+			(at 104.14 133.35 0)
 			(effects
 				(font
@@
 		)
 		(property "Value" "GND"
-			(at 100.33 132.08 0)
+			(at 104.14 132.08 0)
 			(effects
 				(font
@@
 		)
 		(property "Footprint" ""
-			(at 100.33 127 0)
+			(at 104.14 127 0)
 			(effects
 				(font
@@
 		)
 		(property "Datasheet" ""
-			(at 100.33 127 0)
+			(at 104.14 127 0)
 			(effects
 				(font
@@
 		)
 		(property "Description" "Power symbol creates a global label with name \"GND\" , ground"
-			(at 100.33 127 0)
+			(at 104.14 127 0)
 			(effects
 				(font
@@
 	(symbol
 		(lib_id "power:GND")
-		(at 106.68 107.95 0)
+		(at 104.14 107.95 0)
 		(unit 1)
 		(exclude_from_sim no)
@@
 		(fields_autoplaced yes)
 		(property "Reference" "#PWR012"
-			(at 106.68 114.3 0)
+			(at 104.14 114.3 0)
 			(effects
 				(font
@@
 		)
 		(property "Value" "GND"
-			(at 106.68 113.03 0)
+			(at 104.14 113.03 0)
 			(effects
 				(font
@@
 		)
 		(property "Footprint" ""
-			(at 106.68 107.95 0)
+			(at 104.14 107.95 0)
 			(effects
 				(font
@@
 		)
 		(property "Datasheet" ""
-			(at 106.68 107.95 0)
+			(at 104.14 107.95 0)
 			(effects
 				(font
@@
 		)
 		(property "Description" "Power symbol creates a global label with name \"GND\" , ground"
-			(at 106.68 107.95 0)
+			(at 104.14 107.95 0)
 			(effects
 				(font
@@
 	(symbol
 		(lib_id "Connector_Generic:Conn_01x02")
-		(at 93.98 125.73 180)
+		(at 97.79 125.73 180)
 		(unit 1)
 		(exclude_from_sim no)
@@
 		(on_board yes)
 		(dnp no)
-		(fields_autoplaced yes)
 		(property "Reference" "J5"
-			(at 93.98 116.84 0)
+			(at 97.79 116.84 0)
 			(effects
 				(font
@@
 		)
 		(property "Value" "Switch_1"
-			(at 93.98 119.38 0)
+			(at 100.33 119.38 0)
 			(effects
 				(font
@@
 		)
 		(property "Footprint" "Connector_PinHeader_2.54mm:PinHeader_1x02_P2.54mm_Vertical"
-			(at 93.98 125.73 0)
+			(at 97.79 125.73 0)
 			(effects
 				(font
@@
 		)
 		(property "Datasheet" "~"
-			(at 93.98 125.73 0)
+			(at 97.79 125.73 0)
 			(effects
 				(font
@@
 		)
 		(property "Description" "Generic connector, single row, 01x02, script generated (kicad-library-utils/schlib/autogen/connector/)"
-			(at 93.98 125.73 0)
+			(at 97.79 125.73 0)
 			(effects
 				(font
@@
 		)
 		(property "LCSC" "C160388"
-			(at 93.98 125.73 0)
+			(at 97.79 125.73 0)
 			(effects
 				(font
@@
 	(symbol
 		(lib_id "Connector_Generic:Conn_01x02")
-		(at 100.33 106.68 180)
+		(at 97.79 106.68 180)
 		(unit 1)
 		(exclude_from_sim no)
@@
 		(on_board yes)
 		(dnp no)
-		(fields_autoplaced yes)
 		(property "Reference" "J4"
-			(at 100.33 97.79 0)
+			(at 97.79 97.79 0)
 			(effects
 				(font
@@
 		)
 		(property "Footprint" "Connector_PinHeader_2.54mm:PinHeader_1x02_P2.54mm_Vertical"
-			(at 100.33 106.68 0)
+			(at 97.79 106.68 0)
 			(effects
 				(font
@@
 		)
 		(property "Datasheet" "~"
-			(at 100.33 106.68 0)
+			(at 97.79 106.68 0)
 			(effects
 				(font
@@
 		)
 		(property "Description" "Generic connector, single row, 01x02, script generated (kicad-library-utils/schlib/autogen/connector/)"
-			(at 100.33 106.68 0)
+			(at 97.79 106.68 0)
 			(effects
 				(font
@@
 		)
 		(property "LCSC" "C160388"
-			(at 100.33 106.68 0)
+			(at 97.79 106.68 0)
 			(effects
 				(font
@@
 		(on_board yes)
 		(dnp no)
-		(fields_autoplaced yes)
 		(property "Reference" "J7"
 			(at 120.65 97.79 0)
@@
 		)
 		(property "Value" "Switch_1"
-			(at 120.65 100.33 0)
+			(at 123.19 100.33 0)
 			(effects
 				(font
@@
 		(on_board yes)
 		(dnp no)
-		(fields_autoplaced yes)
 		(property "Reference" "J2"
 			(at 120.65 116.84 0)
@@
 		)
 		(property "Value" "Switch_2"
-			(at 120.65 119.38 0)
+			(at 123.19 119.38 0)
 			(effects
 				(font
