File: modbus-pir-2servos/modbus-pir-2servos.kicad_pcb (KiCad board)
At the start: 4 copper layers, 67 x 66 mm, 94 parts, among them J1 USB_B_Micro, J2 Conn_01x02, J4 Conn_02x10_Odd_Even, J5 Conn_01x02, J6 Conn_01x04, M1 Motor_Servo, M2 Motor_Servo, Q2 Q_PMOS_GSD, Q3 MMBT3904, SW1 RESET, SW2 USB_BOOT, U1 SP3485EN, U11 Logo, U2 LMR16030S, U3 RP2040, U4 HT75xx-1-SOT89, U5 PIR_P924M-S, U6 PIR_P924M-S, U7 PCF8563T, U8 LMR14050S, U9 W25Q128JVS, Y1 Crystal_GND24, Y2 Crystal

Commit message: Fix small issues
Parts:
- removed D11, D16: D_Shockley, Diode_SMD:D_SOD-323
- removed JP1: Jumper_3_Open, Connector_PinSocket_2.54mm:PinSocket_1x03_P2.54mm_Vertical
- removed Q3: MMBT3904, Package_TO_SOT_SMD:SOT-23
- added BZ1: Buzzer, cacophony-footprints:BUZ-TH_BD9.0-P5.00-D0.6-FD, F.Cu at (107.8, 87.4)
- added D3: D, Diode_SMD:D_SOD-123F, F.Cu at (156.6, 93.4)
- added H4: MountingHole_Pad, MountingHole:MountingHole_3.2mm_M3_Pad, F.Cu at (99.0, 86.4)
- added J3: Conn_01x05, Connector_JST:JST_XA_B05B-XASK-1-A_1x05_P2.50mm_Vertical, F.Cu at (98.5, 96.8)
- added Q1: 2N7002, Package_TO_SOT_SMD:SOT-23, F.Cu at (108.1, 94.1)
- added SW3: SW_Coded_SH-7010, cacophony-footprints:SW-TH_6P-L10.0-W10.0-P2.54-LS7.6_TSR-10, F.Cu at (138.5, 117.4)
- added SW4: SW_Push_DPDT, cacophony-footprints:SW-TH_K3-2235D-F1, F.Cu at (147.5, 117.6)
- D2: value D_Shockley -> D; footprint Diode_SMD:D_SMA -> Diode_SMD:D_SOD-123F
- J1: footprint cacophony-footprints:920-E52A2021S10100 -> cacophony-footprints:MICRO-USB-TH_MICRO-USB-A14
- J2: footprint Connector_JST:JST_XA_S02B-XASK-1_1x02_P2.50mm_Horizontal -> Connector_JST:JST_XA_B02B-XASK-1-A_1x02_P2.50mm_Vertical
- J4: value Conn_02x10_Odd_Even -> Conn_02x05_Odd_Even; footprint Connector_PinSocket_2.54mm:PinSocket_2x07_P2.54mm_Vertical -> Connector_PinHeader_2.54mm:PinHeader_2x05_P2.54mm_Vertical
- J6: value Conn_01x04 -> Conn_01x02; footprint Connector_JST:JST_XA_S04B-XASK-1_1x04_P2.50mm_Horizontal -> Connector_PinSocket_2.54mm:PinSocket_1x02_P2.54mm_Vertical
- M1, M2: value Motor_Servo -> Servo; footprint Connector_JST:JST_XA_S03B-XASK-1_1x03_P2.50mm_Horizontal -> Connector_JST:JST_XA_B03B-XASK-1-A_1x03_P2.50mm_Vertical
- R1: value 100k -> 10k
- R2: value 100k -> 100R
- moved H3 87.3 mm to (99.0, 146.4)
- moved J4 66.5 mm to (107.9, 110.6), turned to 90 degrees
- moved H2 59.0 mm to (169.0, 86.4)
- moved R6 36.1 mm to (102.7, 142.0), turned to 180 degrees
- moved R1 33.1 mm to (152.8, 93.2)
- moved U5 32.7 mm to (161.7, 103.8), turned to 180 degrees
- moved U11 27.8 mm to (126.3, 129.0)
- moved SW1 26.4 mm to (130.3, 121.5), turned to 90 degrees
- moved R7 25.7 mm to (103.4, 119.4), turned to 180 degrees
- moved H1 23.9 mm to (169.0, 146.4)
- moved C9 23.5 mm to (153.8, 93.2), turned to -90 degrees
- moved C26 23.1 mm to (111.3, 145.4)
- moved M1 22.9 mm to (98.5, 133.0)
- moved M2 22.8 mm to (98.5, 121.8)
- moved D13 22.7 mm to (115.1, 105.2), turned to 0 degrees
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Connections:
- net /SERVO_1 renamed SERVO_1
- net /SERVO_2 renamed SERVO_2
- D2 pad 1: +12V -> Net-(C9-Pad1)
- D2 pad 2: Net-(D2-Pad2) -> +3V3
- J1 pad 1: Net-(D2-Pad2) -> unconnected-(J1-Pad1)
- J4 pad 1: +3V3 -> GND
- J4 pad 10: GND -> /GPIO9
- J4 pad 2: GND -> +3V3
- J4 pad 3: /GPIO17 -> GND
- J4 pad 4: GND -> /GPIO6
- J4 pad 5: /GPIO22 -> /GPIO10
- J4 pad 6: GND -> /GPIO7
- J4 pad 7: /GPIO26_ADC0 -> /GPIO11
- J4 pad 8: GND -> /GPIO8
- J4 pad 9: /GPIO27_ADC1 -> /GPIO12
- J6 pad 1: GND -> ~{RE}
- J6 pad 2: /+ve -> DE
- M1 pad 1: Net-(M1-Pad1) -> GND
- M1 pad 3: GND -> Net-(M1-Pad3)
- M2 pad 1: Net-(M2-Pad1) -> GND
- M2 pad 3: GND -> Net-(M2-Pad3)
- R1 pad 1: TX -> RTC_BAT
- R1 pad 2: Net-(Q3-Pad1) -> Net-(BT1-Pad1)
- R2 pad 1: DE -> Net-(BZ1-Pad2)
- R2 pad 2: +3V3 -> Net-(Q1-Pad3)
- R6 pad 2: Net-(M1-Pad1) -> Net-(M1-Pad3)
- R7 pad 2: Net-(M2-Pad1) -> Net-(M2-Pad3)
- U3 pad 14: 6V_Enable -> /GPIO11
- U3 pad 16: /GPIO13 -> 6V_Enable
- U3 pad 27: /IR_LED_ENABLE -> R_ENC_1
- U3 pad 28: /GPIO17 -> R_ENC_4
- U3 pad 29: /PIR_1 -> R_ENC_2
- U3 pad 30: /PIR_2 -> R_ENC_8
- U3 pad 31: /PIR_3 -> 24_hour
- U3 pad 32: /PIR_4 -> PIR_2
- U3 pad 34: /GPIO22 -> PIR_1
- U3 pad 38: /GPIO26_ADC0 -> RTC_BAT
- U3 pad 4: ~{RE RP2040} -> ~{RE}
- U3 pad 5: unconnected-(U3-Pad5) -> DE
- U3 pad 7: /GPIO5 -> BUZZER
- U5 pad 4: /PIR_1 -> PIR_1
- U6 pad 4: /PIR_2 -> PIR_2
Routing:
- net +12V: track 132.9 -> 57.4 mm, vias 0 -> 2
- net PIR_2: track 0.00 -> 53.2 mm, vias 0 -> 2
- net /GPIO17: track 42.6 -> 0.00 mm, vias 1 -> 0
- net /GPIO26_ADC0: track 41.0 -> 0.00 mm, vias 1 -> 0
- net /GPIO22: track 40.7 -> 0.00 mm, vias 1 -> 0
- net PIR_1: track 0.00 -> 38.8 mm
- net /GPIO27_ADC1: track 38.4 -> 0.00 mm, vias 1 -> 0
- net /GPIO28_ADC2: track 35.8 -> 0.00 mm, vias 1 -> 0
- net /GPIO29_ADC3: track 33.4 -> 0.00 mm, vias 1 -> 0
- net Net-(M1-Pad1): track 33.2 -> 0.00 mm, vias 1 -> 0
- net SERVO_1: track 12.9 -> 42.8 mm
- net RTC_BAT: track 0.00 -> 29.1 mm, vias 0 -> 2
- net 24_hour: track 0.00 -> 23.9 mm
- net /+ve: track 22.6 -> 0.00 mm
- net R_ENC_2: track 0.00 -> 22.2 mm
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- added copper zone on F.Cu, net /+ve
Other:
- board size 67 x 66 mm -> 80 x 70 mm
- board text added: "A"
- board text added: "B"
- board text added: "INT"
- board text removed: "17"
- board text removed: "22"
- board text removed: "26"
- board text removed: "27"
- board text removed: "28"
- board text removed: "29"
- board text removed: "3.3V"
- board text removed: "V0.3.0"

Commit message: Version 1.0.0 of modbus-pir-2servos
Other:
- board text added: "V1.0.0"
Changed lines of the file:
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@@
     (effects (font (size 0.8128 0.8128) (thickness 0.1524)))
   )
-  (gr_text "B" (at 103.125 101.835) (layer "F.SilkS")
+  (gr_text "B" (at 102.8 104.4) (layer "F.SilkS")
     (effects (font (size 0.8128 0.8128) (thickness 0.1524)))
   )
@@
     (effects (font (size 0.8128 0.8128) (thickness 0.1524)))
   )
+  (gr_text "V1.0.0" (at 115 119.2) (layer "F.SilkS")
+    (effects (font (size 2 2) (thickness 0.4)))
+  )
   (gr_text "6V" (at 102.9 124.5) (layer "F.SilkS")
     (effects (font (size 0.8128 0.8128) (thickness 0.1524)))
@@
     (effects (font (size 0.8128 0.8128) (thickness 0.1524)))
   )
-  (gr_text "A" (at 103.125 104.335) (layer "F.SilkS")
+  (gr_text "A" (at 102.8 101.8) (layer "F.SilkS")
     (effects (font (size 0.8128 0.8128) (thickness 0.1524)))
   )
@@
     )
   )
-  (group "" (id a889fece-ee7b-4c74-b079-91fe11f515c8)
-    (members
-      1649b09a-2ad6-4a2b-931f-e061a6b5852b
-      38932013-27ef-41f7-8c8a-35d810841ed3
-      b0de5629-15b4-4ae6-b92e-c88bb0f3c98b
-      b54ed3aa-5c56-4492-a9f9-0de029e51696
-      b7debfe0-229e-46f8-83a1-8f18faa81fbb
-      d30f7b74-ff79-4adf-8c62-eb9dab24d587
-    )
-  )

Commit message: WIP
Parts:
- removed BT1: Battery_Cell, cacophony-footprints:CR1220
- removed C1: 220uF, cacophony-footprints:CAP-SMD_BD8.0-L8.3-W8.3-LS9.3-FD
- removed C2, C3: 2.2uF, Capacitor_SMD:C_0805_2012Metric
- removed C24, C8: 47uF, Capacitor_SMD:C_1206_3216Metric
- removed C4: 470nF, Capacitor_SMD:C_0603_1608Metric
- removed C5: 10nF, Capacitor_SMD:C_0402_1005Metric
- removed C6: 100nF, Capacitor_SMD:C_0603_1608Metric
- removed C7: 1uF, Capacitor_SMD:C_0402_1005Metric
- removed D1: D_Shockley, Diode_SMD:D_SMA
- removed D12: D_Zener, Diode_SMD:D_MiniMELF
- removed D3: D, Diode_SMD:D_SOD-123F
- removed L1: 15uH, cacophony-footprints:IND-SMD_L6.0-W6.0_SWPA6045S
- removed Q2: Q_PMOS_GSD, Package_TO_SOT_SMD:SOT-23
- removed R14: 33k, Resistor_SMD:R_0603_1608Metric
- removed R15: 100k, Resistor_SMD:R_0603_1608Metric
- removed R16: 270k, Resistor_SMD:R_0603_1608Metric
- removed R5: 47k, Resistor_SMD:R_0402_1005Metric
- removed U2: LMR16030S, Package_SO:TI_SO-PowerPAD-8
- added BT2: Battery_Cell, cacophony-library:CAP-SMD_FL11E, F.Cu at (60.4, 10.4)
- added C1001: 22uF, Capacitor_SMD:C_0805_2012Metric, F.Cu at (73.7, 51.4)
- added C1002: 22uF, Capacitor_SMD:C_0805_2012Metric, F.Cu at (73.7, 49.4)
- added C1003: 2.2uF, Capacitor_SMD:C_0402_1005Metric, F.Cu at (74.1, 48.0)
- added C1004: 10uF, Capacitor_SMD:C_0402_1005Metric, F.Cu at (74.1, 43.0)
- added C1005: 22uF, Capacitor_SMD:C_0603_1608Metric, F.Cu at (73.8, 41.8)
- added C1006: 22uF, Capacitor_SMD:C_0603_1608Metric, F.Cu at (73.8, 40.4)
- added C1007: 22uF, Capacitor_SMD:C_0603_1608Metric, F.Cu at (73.8, 38.9)
- added C1008: 22uF, Capacitor_SMD:C_0603_1608Metric, F.Cu at (73.8, 37.5)
- added C1009: 100nF, Capacitor_SMD:C_0402_1005Metric, F.Cu at (77.2, 44.5)
- added C25: 47uF, Capacitor_SMD:C_1206_3216Metric, F.Cu at (5.36, 46.3)
- added C35: 47uF, Capacitor_SMD:C_1206_3216Metric, F.Cu at (7.66, 46.3)
- added C36: 47uF, Capacitor_SMD:C_1206_3216Metric, F.Cu at (9.96, 46.3)
- added C37: 47uF, Capacitor_SMD:C_1206_3216Metric, F.Cu at (5.34, 51.7)
- added C38: 22pF, Capacitor_SMD:C_0402_1005Metric, F.Cu at (69.4, 3.56)
- added C39: 100n, Capacitor_SMD:C_0402_1005Metric, F.Cu at (46.7, 56.7)
- added C40: 1uF, Capacitor_SMD:C_0402_1005Metric, F.Cu at (38.9, 57.8)
- added C41: 1uF, Capacitor_SMD:C_0402_1005Metric, F.Cu at (44.9, 57.8)
- added D4: D, Diode_SMD:D_SOD-523, F.Cu at (50.7, 19.1)
- added FB1001: FerriteBead, Inductor_SMD:L_0805_2012Metric, F.Cu at (73.5, 35.5)
- added J10: Conn_01x02, Connector_PinHeader_2.00mm:PinHeader_1x02_P2.00mm_Vertical, F.Cu at (54.8, 12.7)
- added J7: Switch_1, cacophony-library:JST_SH_BM02B-SRSS-TB_1x02-1MP_P1.00mm_Vertical, F.Cu at (60.1, 56.0)
- added J8: Conn_02x03_Odd_Even, Connector_PinHeader_2.54mm:PinHeader_2x03_P2.54mm_Vertical, F.Cu at (51.3, 12.7)
- added J9: Conn_01x08, Connector_JST:JST_XA_S08B-XASK-1_1x08_P2.50mm_Horizontal, B.Cu at (20.6, 11.3)
- added JP1: SolderJumper_2_Bridged, Jumper:SolderJumper-2_P1.3mm_Bridged_RoundedPad1.0x1.5mm, F.Cu at (57.6, 10.4)
- added L1001: INDUCTOR, Inductor_SMD:L_1008_2520Metric, F.Cu at (72.0, 45.5)
- added Q3: Q_PMOS_GSD, Package_TO_SOT_SMD:SOT-23, F.Cu at (11.5, 23.5)
- added Q4: 2N7002, Package_TO_SOT_SMD:SOT-23, F.Cu at (11.5, 27.4)
- added Q5: Q_PMOS_GSD, Package_TO_SOT_SMD:SOT-23, F.Cu at (11.3, 35.0)
- added Q6: 2N7002, Package_TO_SOT_SMD:SOT-23, F.Cu at (11.3, 38.9)
- added R1001: 470k, Resistor_SMD:R_0402_1005Metric, F.Cu at (76.2, 42.1)
- added R1002: 10k, Resistor_SMD:R_0402_1005Metric, F.Cu at (77.2, 47.8)
- added R1003: 150k, Resistor_SMD:R_0402_1005Metric, F.Cu at (76.3, 43.0)
- added R1004: 100k, Resistor_SMD:R_0402_1005Metric, F.Cu at (76.2, 41.1)
- added R13: 1k, Resistor_SMD:R_0402_1005Metric, F.Cu at (23.8, 19.2)
- added R21: 1k, Resistor_SMD:R_0402_1005Metric, F.Cu at (46.6, 18.9)
- added R23: 1k, Resistor_SMD:R_0402_1005Metric, F.Cu at (56.9, 7.30)
- added R24: 10k, Resistor_SMD:R_0402_1005Metric, F.Cu at (13.7, 26.1)
- added R28: 1k, Resistor_SMD:R_0402_1005Metric, F.Cu at (46.6, 20.4)
- added R29: 10k, Resistor_SMD:R_0402_1005Metric, F.Cu at (13.5, 37.9)
- added R30: 1k, Resistor_SMD:R_0402_1005Metric, F.Cu at (30.4, 24.3)
- added R31: 1k, Resistor_SMD:R_0402_1005Metric, F.Cu at (32.8, 18.9)
- added R32: 27k, Resistor_SMD:R_0603_1608Metric, F.Cu at (46.9, 57.9)
- added R33: 1k, Resistor_SMD:R_0402_1005Metric, F.Cu at (32.8, 20.8)
- added R34: 1k, Resistor_SMD:R_0402_1005Metric, F.Cu at (60.8, 51.9)
- added R35: 1k, Resistor_SMD:R_0402_1005Metric, F.Cu at (32.1, 28.3)
- added SW5: SW_Push_DPDT, cacophony-library:SW-TH_K3-2235D-F1, F.Cu at (43.0, 49.6)
- added TP1001: TestPoint_2Pole, cacophony-library:test-point-2p, F.Cu at (73.5, 33.4)
- added U1001: TPS63070RNMR, cacophony-library:TPS63070, F.Cu at (75.1, 45.5)
- BZ1: footprint cacophony-footprints:BUZ-TH_BD9.0-P5.00-D0.6-FD -> cacophony-library:BUZ-TH_BD9.0-P5.00-D0.6-FD
- C10, C15: value 1u -> 1uF
- C26: footprint cacophony-footprints:CAP-SMD_BD8.0-L8.3-W8.3-LS9.3-FD -> cacophony-library:CAP-SMD_BD8.0-L8.3-W8.3-LS9.3-FD
- C27, C28: value 2.2uF -> 22uF
- C32: value 1uF -> 22pF
- H1, H2, H3, H4: footprint MountingHole:MountingHole_3.2mm_M3_Pad -> cacophony-library:MountingHole_3.2mm_M3
- J1: footprint cacophony-footprints:MICRO-USB-TH_MICRO-USB-A14 -> cacophony-library:MICRO-USB-TH_MICRO-USB-A14
- J2: value Conn_01x02 -> Switch_2; footprint Connector_JST:JST_XA_B02B-XASK-1-A_1x02_P2.50mm_Vertical -> cacophony-library:JST_SH_BM02B-SRSS-TB_1x02-1MP_P1.00mm_Vertical
- J3: value Conn_01x05 -> Conn_02x03_Odd_Even; footprint Connector_JST:JST_XA_B05B-XASK-1-A_1x05_P2.50mm_Vertical -> Connector_PinHeader_2.54mm:PinHeader_2x03_P2.54mm_Vertical
- J4: value Conn_02x05_Odd_Even -> Switch_1; footprint Connector_PinHeader_2.54mm:PinHeader_2x05_P2.54mm_Vertical -> Connector_PinHeader_2.54mm:PinHeader_1x02_P2.54mm_Vertical
- J5: value Conn_01x02 -> Switch_1; footprint Connector_PinSocket_2.54mm:PinSocket_1x02_P2.54mm_Vertical -> Connector_PinHeader_2.54mm:PinHeader_1x02_P2.54mm_Vertical
- J6: value Conn_01x02 -> SWD; footprint Connector_PinSocket_2.54mm:PinSocket_1x02_P2.54mm_Vertical -> Connector_PinHeader_2.54mm:PinHeader_1x03_P2.54mm_Vertical
- L2: footprint cacophony-footprints:IND-SMD_L7.0-W6.6 -> cacophony-library:IND-SMD_L7.0-W6.6
- R1: value 10k -> 1k
- R18: value 10K -> 10k
- R19: value 100k -> 1k
- R20: value 120R -> 1k
- R22, R6, R7, R9: value 1K -> 1k
- R3, R4: value 27R -> 33ohm; footprint Resistor_SMD:R_0603_1608Metric -> Resistor_SMD:R_0402_1005Metric
- R8: value 82K -> 27k
- RV1: value R_Potentiometer -> 10k
- SW3: footprint cacophony-footprints:SW-TH_6P-L10.0-W10.0-P2.54-LS7.6_TSR-10 -> cacophony-library:SW-TH_6P-L10.0-W10.0-P2.54-LS7.6_TSR-10
- SW4: footprint cacophony-footprints:SW-TH_K3-2235D-F1 -> cacophony-library:SW-TH_K3-2235D-F1
- U1: value SP3485EN -> TPL0401B-10-Q1; footprint Package_SO:SOIC-8_3.9x4.9mm_P1.27mm -> Package_TO_SOT_SMD:Texas_R-PDSO-G6
- U11: footprint cacophony-footprints:logo -> cacophony-library:logo
- U3: footprint cacophony-footprints:RP2040-QFN-56 -> cacophony-library:RP2040-QFN-56
- U5, U6: footprint cacophony-footprints:PIR_P924M-S -> cacophony-library:PIR_P924M-S
- moved H2 165.4 mm to (5.00, 65.0)
- moved U5 151.3 mm to (27.0, 35.0), turned to -90 degrees
- moved R1 148.2 mm to (23.8, 20.2), turned to 0 degrees
- moved U6 144.3 mm to (53.0, 35.0), turned to 0 degrees
- moved M1 143.6 mm to (5.61, 23.5)
- moved H3 143.4 mm to (75.0, 5.00)
- moved C28 139.1 mm to (5.69, 56.9), turned to 90 degrees
- moved C32 136.6 mm to (69.4, 5.42), turned to 90 degrees
- moved C27 136.2 mm to (7.65, 56.9), turned to 90 degrees
- moved C34 136.0 mm to (7.64, 51.7), turned to -90 degrees
- moved U4 134.7 mm to (42.0, 55.8), turned to 90 degrees
- moved C29 133.6 mm to (9.36, 57.1), turned to 90 degrees
- moved R25 133.2 mm to (10.9, 61.9), turned to 180 degrees
- moved D2 133.0 mm to (59.6, 7.54)
- moved RV1 132.7 mm to (51.0, 56.0), turned to 90 degrees
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Connections:
- net /SW_6V renamed /power/SW_6V
- net Net-(C9-Pad1) renamed /RTC_V_{DD}
- net Net-(R9-Pad2) renamed /USB_BOOT
- C32 pad 1: +6V -> Net-(U7-OSCI)
- D13 pad 1: Net-(D13-Pad1) -> GND
- D13 pad 2: Net-(D13-Pad2) -> Net-(D13-A)
- J2 pad 2: /+ve -> SWITCH_2
- J3 pad 2: /+ve -> /GPIO13
- J3 pad 3: /RS485_A -> GND
- J3 pad 4: /RS485_B -> /GPIO14
- J3 pad 5: /INTERRUPT -> +3V3
- J4 pad 2: +3V3 -> SWITCH_1
- J5 pad 1: /SWD -> GND
- J5 pad 2: /SWCLK -> SWITCH_2
- J6 pad 1: ~{RE} -> /SWD
- J6 pad 2: DE -> GND
- M1 pad 2: +6V -> Net-(M1-+Ve)
- M1 pad 3: Net-(M1-Pad3) -> SERVO_1
- M2 pad 2: +6V -> Net-(M2-+Ve)
- M2 pad 3: Net-(M2-Pad3) -> SERVO_2
- R1 pad 1: RTC_BAT -> SERVO_1
- R1 pad 2: Net-(BT1-Pad1) -> /SERVO_1_PHY
- R19 pad 1: Net-(D12-Pad2) -> Net-(U3-GPIO10)
- R19 pad 2: GND -> SWITCH_2
- R20 pad 1: /RS485_A -> /SERVO_2_PHY
- R20 pad 2: /RS485_B -> SERVO_2_EN
- R22 pad 1: GND -> Net-(D13-A)
- R22 pad 2: Net-(D13-Pad1) -> LED_1_PHY
- R25 pad 2: 6V_Enable -> 6V_EN
- R3 pad 1: /USB_D+ -> /USB_PHY_D+
- R3 pad 2: Net-(R3-Pad2) -> /USB_D+
- R4 pad 1: /USB_D- -> /USB_PHY_D-
- R4 pad 2: Net-(R4-Pad2) -> /USB_D-
- R6 pad 1: SERVO_1 -> PIR_2
- R6 pad 2: Net-(M1-Pad3) -> /input-output/PIR_2_PHY
- R7 pad 1: SERVO_2 -> PIR_1
- R7 pad 2: Net-(M2-Pad3) -> /input-output/PIR_1_PHY
- R8 pad 1: Net-(R8-Pad1) -> +3V3_Lin
- R8 pad 2: Net-(R8-Pad2) -> /input-output/PIR_SENS_POT_MANUAL
- RV1 pad 2: Net-(R8-Pad2) -> /input-output/PIR_SENS_POT_MANUAL
- SW4 pad 2: 24_hour -> NIGHT_ONLY
- U1 pad 1: RX -> +3V3_Lin
- U1 pad 2: ~{RE} -> GND
- U1 pad 3: DE -> SCL
- U1 pad 4: TX -> SDA
- U1 pad 5: GND -> /input-output/PIR_SENS_POT_PROG
- U1 pad 6: /RS485_A -> unconnected-(U1-H-Pad6)
- U3 pad 11: /GPIO8 -> /6V_EN_PHY
- U3 pad 12: /GPIO9 -> Net-(U3-GPIO9)
- U3 pad 13: /GPIO10 -> Net-(U3-GPIO10)
- U3 pad 14: /GPIO11 -> Net-(U3-GPIO11)
- U3 pad 15: /GPIO12 -> PIR_1
- U3 pad 16: 6V_Enable -> /GPIO13
- U3 pad 17: SERVO_2 -> /GPIO14
- U3 pad 18: SERVO_1 -> /GPIO15
- U3 pad 2: TX -> /RP2040_TX_IN_PHY
- U3 pad 27: R_ENC_1 -> PIR_2
- U3 pad 28: R_ENC_4 -> BUZZER
- U3 pad 3: RX -> RP2040_RX_IN
- U3 pad 30: R_ENC_8 -> R_ENC_4
- U3 pad 31: 24_hour -> R_ENC_8
- U3 pad 32: PIR_2 -> R_ENC_1
- U3 pad 34: PIR_1 -> NIGHT_ONLY
- U3 pad 38: RTC_BAT -> /PIR_SENS_POT_FB
- U3 pad 4: ~{RE} -> /SERVO_1_EN_PHY
- U3 pad 41: /GPIO29_ADC3 -> /RTC_BAT_SENSE_PHY
- U3 pad 46: Net-(R4-Pad2) -> /USB_PHY_D-
- U3 pad 47: Net-(R3-Pad2) -> /USB_PHY_D+
- U3 pad 5: DE -> /SERVO_1_PHY
- U3 pad 6: Net-(D13-Pad2) -> /RP2040_TX_OUT_PHY
- U3 pad 7: BUZZER -> RP2040_RX_OUT
- U3 pad 8: /GPIO6 -> LED_1_PHY
- U3 pad 9: /GPIO7 -> /SERVO_2_PHY
- U4 pad 3: Net-(R8-Pad1) -> +3V3_Lin
- U5 pad 2: Net-(R8-Pad2) -> PIR_SENS_POT
- U5 pad 3: Net-(R8-Pad1) -> +3V3_Lin
- U5 pad 4: PIR_1 -> /input-output/PIR_1_PHY
- U6 pad 2: Net-(R8-Pad2) -> PIR_SENS_POT
- U6 pad 3: Net-(R8-Pad1) -> +3V3_Lin
- U6 pad 4: PIR_2 -> /input-output/PIR_2_PHY
- U7 pad 1: Net-(U7-Pad1) -> Net-(U7-OSCI)
- U8 pad 3: 6V_Enable -> 6V_EN
- Y2 pad 2: Net-(U7-Pad1) -> Net-(U7-OSCI)
Routing:
- net Net-(U3-GPIO9): track 0.00 -> 65.4 mm, vias 0 -> 2
- net PIR_SENS_POT: track 0.00 -> 64.4 mm, vias 0 -> 2
- net Net-(U3-GPIO10): track 0.00 -> 63.3 mm, vias 0 -> 2
- net 6V_EN: track 0.00 -> 62.5 mm, vias 0 -> 2
- net +3V3_Lin: track 0.00 -> 58.1 mm, vias 0 -> 1
- net SDA: track 36.0 -> 84.0 mm, vias 0 -> 4
- net PIR_2: track 53.2 -> 7.68 mm, vias 2 -> 0
- net Net-(R8-Pad1): track 43.8 -> 0.00 mm
- net SCL: track 34.0 -> 77.1 mm
- net +12V: track 57.4 -> 14.4 mm, vias 2 -> 26
- net Net-(R8-Pad2): track 38.6 -> 0.00 mm
- net 6V_Enable: track 33.9 -> 0.00 mm, vias 2 -> 0
- net PIR_1: track 38.8 -> 7.55 mm
- net /GPIO13: track 0.00 -> 30.7 mm
- net SERVO_2_EN: track 0.00 -> 30.4 mm
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- added copper zone on In2.Cu, net +12V
- added copper zone on In2.Cu, net +6V
- added copper zone on F.Cu, net /power/3V3_L1
- added copper zone on F.Cu, net /power/3V3_L2
- added copper zone on F.Cu, net /power/3V3_PHY
- added copper zone on B.Cu, net GND
- removed copper zone on B.Cu, net (none)
- removed copper zone on F.Cu, net /+ve
- removed copper zone on F.Cu, net /SW_3V3
Other:
- outline, holes or cut-outs redrawn
- board text added: "${TAG}"
- board text added: "13"
- board text added: "14"
- board text added: "15"
- board text added: "27"
- board text added: "28"
- board text added: "3V3"
- board text added: "GND"
- board text added: "Manual"
- board text added: "Night And Day"
- board text added: "Night Only"
- board text added: "Prog"
- board text added: "RP_RX_IN"
- board text added: "RP_RX_OUT"
- board text added: "RP_TX_IN"
- board text added: "RP_TX_OUT"
- board text added: "SWCLK"
- board text added: "SWD"
- board text removed: "A"
- board text removed: "B"
- board text removed: "INT"
- board text removed: "V1.0.0"

Commit message: WIP
Parts:
- added REF**: Tab, kikit:Tab, F.Cu at (12.0, -0.55)
- added REF**: Tab, kikit:Tab, F.Cu at (12.0, 70.5)
- added REF**: Tab, kikit:Tab, F.Cu at (-0.55, 55.0)
- added REF**: Tab, kikit:Tab, F.Cu at (-0.55, 35.0)
- added REF**: Tab, kikit:Tab, F.Cu at (40.0, 8.45)
- added REF**: Tab, kikit:Tab, F.Cu at (40.0, 60.5)
- added REF**: Tab, kikit:Tab, F.Cu at (80.5, 55.0)
- added REF**: Tab, kikit:Tab, F.Cu at (69.0, -0.55)
- added REF**: Tab, kikit:Tab, F.Cu at (68.0, 70.5)
- added REF**: Tab, kikit:Tab, F.Cu at (80.5, 35.0)
- added REF**: Tab, kikit:Tab, F.Cu at (80.5, 15.0)
- added REF**: Tab, kikit:Tab, F.Cu at (-0.55, 15.0)
